File: kicad/SXMainBoard/SXMainBoard.kicad_pcb (KiCad board)
At the start: 4 copper layers, 243.8 x 243.8 mm, 53 parts, among them J1 PCIE-098-02-X-D-TH, J10 Conn_01x16, J11 Conn_01x16, J12 Conn_01x06, J13 Conn_01x03, J2 Conn_02x03_Odd_Even, J3 ATX24RH, J4 Conn_01x16, J41 CONN_04JST-PTH, J42 CONN_04JST-PTH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

Commit message: Start working on v2 of the micro atx
Parts:
- removed SW1: SW_Push_Dual, Button_Switch_THT:SW_PUSH_6mm
- H1, H2, H3, H4, H5, H6, H7, H8, H9: renamed from REF**; value MountingHole_3.7mm -> MountingHole; footprint Mounting_Holes:MountingHole_3.7mm -> MountingHole:MountingHole_3.7mm
- moved J13 20.3 mm to (108.9, 107.9), turned to 270 degrees
- moved J8 15.6 mm to (108.9, 103.9), turned to 270 degrees
Connections:
- net -12V renamed Net-(J3-Pad14)
- J1 pad A1: /VCC11 -> +5V
- J1 pad A11: /VCC11 -> +5V
- J1 pad A3: /VCC11 -> +5V
- J1 pad A5: /VCC11 -> +5V
- J1 pad A7: /VCC11 -> +5V
- J1 pad A9: /VCC11 -> +5V
- J1 pad B1: /VCC0 -> +5V
- J1 pad B11: /VCC0 -> +5V
- J1 pad B3: /VCC0 -> +5V
- J1 pad B5: /VCC0 -> +5V
- J1 pad B7: /VCC0 -> +5V
- J1 pad B9: /VCC0 -> +5V
- J2 pad 5: Net-(J2-Pad5) -> /~RESET
- J2 pad 6: Net-(J2-Pad6) -> GNDREF
- J3 pad 22: /VCC0 -> +5V
- J3 pad 23: /VCC11 -> +5V
Routing:
- net +5V: track 596.3 -> 0.00 mm
- net /SCK: track 435.4 -> 0.00 mm
- net /A12: track 432.8 -> 0.00 mm
- net +12V: track 423.1 -> 9.72 mm
- net /MEGA_ACTIVE: track 403.4 -> 0.00 mm
- net /MISO: track 374.7 -> 0.00 mm, vias 1 -> 0
- net /A10: track 369.3 -> 0.00 mm
- net /SDA: track 366.3 -> 0.00 mm
- net /PSU_STANDBY: track 328.1 -> 0.00 mm
- net /POWER_OK: track 326.8 -> 0.00 mm
- net /MOSI: track 322.5 -> 0.00 mm, vias 1 -> 0
- net /AD14: track 332.1 -> 20.7 mm
- net /A14: track 286.1 -> 0.00 mm
- net /A31: track 284.2 -> 0.00 mm
- net /A13: track 283.6 -> 0.00 mm
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- removed copper zone on In1.Cu, net +3V3
- removed copper zone on F.Cu, net +5V
- removed copper zone on B.Cu, net GNDREF
Other:
- board text added: "i960Sx "Hanekawa" Main Board (C) 2020 Joshua Scoggins REV 4"
- board text removed: "i960Sx "Hanekawa" Main Board (C) 2020 Joshua Scoggins REV 3"
