File: kicad/i960SxBreakoutBoard/i960SxBreakoutBoard.kicad_pcb (KiCad board)
At the start: 4 copper layers, 100.2 x 110.5 mm, 16 parts, among them J1 PCIE-098-02-X-D-TH, U1 80960Sx, X1 OCXO-14

Commit message: Remove blind vias from the breakout board as AISLER does not support them
Routing:
- net +5V: track 143.6 -> 228.1 mm, vias 6 -> 19
- net /INT0: track 96.5 -> 177.4 mm, vias 1 -> 0
- net /INT1: track 95.8 -> 168.5 mm
- net /INT2: track 101.1 -> 168.7 mm, vias 1 -> 0
- net /DTR: track 91.4 -> 156.6 mm
- net /DEN_: track 100.1 -> 160.7 mm
- net /INT3: track 98.6 -> 158.4 mm
- net /WR: track 111.3 -> 168.7 mm, vias 1 -> 0
- net /HLDA: track 100.7 -> 154.2 mm, vias 1 -> 0
- net /LOCK_: track 143.3 -> 192.9 mm
- net /HOLD: track 104.9 -> 144.1 mm, vias 1 -> 0
- net /A3: track 104.6 -> 69.6 mm
- net /A2: track 103.6 -> 72.9 mm, vias 1 -> 0
- net GND: track 221.9 -> 246.3 mm, vias 18 -> 19
- net /AS_: track 103.8 -> 123.7 mm, vias 3 -> 0
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- added copper zone on In1.Cu, net +5V
- added copper zone on In2.Cu, net GND
- removed copper zone on F.Cu, net +5V
- removed copper zone on B.Cu, net GND
- removed copper zone on In1.Cu, net GND
Other:
- board text added: "80960Sx Interface Board via PCI Express x8 (C) 2020 Joshua Scoggins REV 2"
- board text removed: "80960Sx Interface Board via PCI Express x8 (C) 2020 Joshua Scoggins REV 1"

Commit message: More changes
Parts:
- added D1: POWER LED, LED_THT:LED_D5.0mm, F.Cu at (55.7, 153.5)
- added R2: 330, Resistor_SMD:R_0805_2012Metric_Pad1.15x1.40mm_HandSolder, F.Cu at (63.1, 151.2)
- R1: value 1K -> 910
- moved C12 94.0 mm to (13.7, 92.1)
- moved C8 78.2 mm to (20.1, 102.3)
- moved C2 74.2 mm to (10.1, 107.1)
- moved C3 74.2 mm to (5.01, 107.1)
- moved C1 72.3 mm to (34.4, 92.0)
- moved C10 72.3 mm to (35.6, 65.3)
- moved C11 72.3 mm to (35.9, 74.4)
- moved C4 72.3 mm to (-8.56, 87.4)
- moved C5 72.3 mm to (-8.83, 79.5)
- moved C6 72.3 mm to (3.11, 58.7)
- moved C7 72.3 mm to (6.41, 58.7)
- moved C9 72.3 mm to (16.6, 57.7)
- moved R1 72.3 mm to (0.06, 58.7)
- moved U1 42.6 mm to (97.5, 125.0), turned to 270 degrees
Routing:
- net /LOCK_: track 192.9 -> 0.00 mm
- net /INT0: track 177.4 -> 0.00 mm
- net /INT2: track 168.7 -> 0.00 mm
- net /INT1: track 168.5 -> 0.00 mm, vias 1 -> 0
- net /DEN_: track 160.7 -> 0.00 mm, vias 1 -> 0
- net /INT3: track 158.4 -> 0.00 mm, vias 1 -> 0
- net /DTR: track 156.6 -> 0.00 mm, vias 1 -> 0
- net GND: track 246.3 -> 93.1 mm, vias 19 -> 6
- net +5V: track 228.1 -> 93.3 mm, vias 19 -> 7
- net /A31: track 140.6 -> 64.4 mm
- net /CLK2: track 113.1 -> 186.8 mm
- net /WR: track 168.7 -> 98.5 mm, vias 0 -> 1
- net /HLDA: track 154.2 -> 85.3 mm, vias 0 -> 1
- net /A30: track 128.5 -> 62.3 mm, vias 1 -> 0
- net /HOLD: track 144.1 -> 78.1 mm, vias 0 -> 1
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- removed copper zone on In1.Cu, net +5V
- removed copper zone on In2.Cu, net GND
